Commit message: urdf parse materials added and example load urdf completed

File: examples/crane_robot.urdf (robot description, URDF)
Before this commit: robot origins, 4 links, 3 joints
Links:
- link base: geometry collision box size=0.5 0.5 0.1; visual box size=0.5 0.5 0.1
- link jib: geometry collision box size=1.0 0.1 0.1; visual box size=1.0 0.1 0.1
- link tower: geometry collision box size=0.1 0.1 1.0; visual box size=0.1 0.1 1.0
- link trolley: geometry collision box size=0.15 0.15 0.2; visual sphere radius=0.07
